File: hardware/Radioberry.kicad_pcb (KiCad board)
At the start: 4 copper layers, 65 x 56 mm, 143 parts, among them CN301 DNI, CN302 PINHEAD_PINHD-2X20, IC201 LD1117S25, IC202 LD1117S33, IC203 LD1117S33, IC204 LD1117S12, IC401 AD9866, T401 1:1, T402 8:1, U1 FPGA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

Commit message: radioberry v2.0 beta2
Parts:
- added R307: DNI, hermeslite:SMD-0603, B.Cu at (128.0, 119.5)
- added R308: DNI, hermeslite:SMD-0603, B.Cu at (130.0, 119.5)
- moved R303 3.78 mm to (123.8, 119.5)
- moved R305 0.20 mm to (132.2, 119.5)
- moved R306 0.16 mm to (134.2, 119.5)
- moved R304 0.10 mm to (125.8, 119.5)
Connections:
- net /Frontend/RXEN renamed RXEN
- C216 pad 1: 3V3B -> +2V5
- CN301 pad 13: /GPIO/IO-11 -> IO-11
- CN301 pad 14: /GPIO/IO-12 -> IO-12
- CN302 pad 1: Net-(CN302-Pad1) -> 3V3Rpi
- CN302 pad 9: Net-(CN302-Pad9) -> GND
- FB401 pad 1: Net-(FB401-Pad1) -> 3V3Rpi
- IC204 pad 3: 3V3B -> +2V5
- U1 pad 114: Net-(U1-Pad114) -> /Frontend/RESET
- U1 pad 115: Net-(U1-Pad115) -> IO-14
- U1 pad 119: IO-14 -> IO-13
- U1 pad 120: IO-13 -> IO-12
- U1 pad 121: /GPIO/IO-12 -> IO-11
- U1 pad 125: /GPIO/IO-11 -> IO-10
- U1 pad 132: IO-10 -> IO-09
- U1 pad 133: IO-09 -> IO-08
- U1 pad 134: IO-08 -> +1V2
- U1 pad 61: /Frontend/RESET -> +1V2
Routing:
- net 3V3B: track 153.7 -> 51.9 mm, vias 3 -> 1
- net GND: track 710.4 -> 773.1 mm
- net 3V3Rpi: track 0.00 -> 30.6 mm, vias 0 -> 1
- net +2V5: track 107.2 -> 131.0 mm, vias 1 -> 2
- net IO-12: track 0.00 -> 23.4 mm
- net /Frontend/RESET: track 33.2 -> 53.4 mm, vias 0 -> 2
- net /GPIO/IO-12: track 17.8 -> 0.00 mm
- net IO-11: track 0.00 -> 16.7 mm
- net /GPIO/IO-11: track 15.0 -> 0.00 mm
- net +5V: track 147.9 -> 156.4 mm, vias 3 -> 2
- net +1V2: track 202.7 -> 208.8 mm, vias 10 -> 11
- net +3V3: track 191.1 -> 188.0 mm
- net IO-10: track 24.7 -> 23.4 mm
- net GPIO11: track 52.4 -> 51.3 mm
- net IO-14: track 24.1 -> 23.5 mm
Other:
- board text added: "Radioberry V2.0 beta2"
- board text removed: "Radioberry V2.0 beta1"
