File: hardware/Radioberry.kicad_pcb (KiCad board)
At the start: 4 copper layers, 65 x 56 mm, 146 parts, among them CN301 DNI, CN302 PINHEAD_PINHD-2X20, IC201 LD1117S25, IC202 LD1117S33, IC203 LD1117S33, IC204 LD1117S12, IC401 AD9866, T401 1:1, T402 8:1, U1 FPGA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

Commit message: beta version silk at bottom updated
Other:
- board text added: "Radioberry V2.0 beta3"
- board text removed: "Radioberry V2.0 beta2"
- board text removed: "beta3"
Changed lines of the file:
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@@
     (area 82.508399 70.949999 200.918338 151.78355)
     (thickness 1.6)
-    (drawings 12)
+    (drawings 11)
     (tracks 1510)
     (zones 0)
@@
     (1 In1.Cu signal hide)
     (2 In2.Cu signal hide)
-    (31 B.Cu signal hide)
+    (31 B.Cu signal)
     (32 B.Adhes user hide)
     (33 F.Adhes user hide)
-    (34 B.Paste user hide)
+    (34 B.Paste user)
     (35 F.Paste user)
-    (36 B.SilkS user hide)
+    (36 B.SilkS user)
     (37 F.SilkS user)
     (38 B.Mask user hide)
@@
       (drillshape 0)
       (scaleselection 1)
-      (outputdirectory release/beta3/position/))
+      (outputdirectory release/beta3/pcb/))
   )
   (net 0 "")
@@
     )
   )
-  (gr_text beta3 (at 100.2 124.6) (layer F.SilkS)
-    (effects (font (size 1 1) (thickness 0.25)))
-  )
   (gr_arc (start 154 72) (end 154 71) (angle 90) (layer Edge.Cuts) (width 0.1))
   (gr_arc (start 154 126) (end 155 126) (angle 90) (layer Edge.Cuts) (width 0.1))
@@
   (gr_line (start 155 72) (end 155 126) (angle 90) (layer Edge.Cuts) (width 0.1))
   (gr_line (start 91 71) (end 154 71) (angle 90) (layer Edge.Cuts) (width 0.1))
-  (gr_text "Radioberry V2.0 beta2" (at 127.73 81.06) (layer B.SilkS)
+  (gr_text "Radioberry V2.0 beta3" (at 127.73 81.06) (layer B.SilkS)
     (effects (font (size 1.5 1.5) (thickness 0.3)) (justify mirror))
   )

Commit message: beta4
Connections:
- net RXEN renamed /Frontend/RXEN
- U1 pad 118: GND -> Net-(U1-Pad118)
- U1 pad 53: (no net) -> /Frontend/CLKOUT1
Routing:
- net /Frontend/CLKOUT1: track 21.2 -> 35.8 mm, vias 0 -> 2
Other:
- board text added: "Radioberry V2.0 beta4"
- board text removed: "Radioberry V2.0 beta3"
