File: hardware/Radioberry-Frontend.sch (KiCad schematic (older format))
At the start: 56 parts, among them IC401 AD9866, T401 1:1, T402 8:1, U1 FPGA, X400 TCXO, X401 SMA, X402 SMA

Commit message: radioberry v2.0 beta2
Connections:
- net 3V3Rpi: now reaches FB401.1
Changed lines of the file:
@@
 LIBS:Radioberry
 LIBS:hermeslite
+LIBS:power
 LIBS:Radioberry-cache
 EELAYER 25 0
@@
 $EndComp
 $Comp
-L GND #PWR043
+L GND #PWR047
 U 1 1 59CDDAE7
 P 5925 8425
-F 0 "#PWR043" H 5925 8175 50  0001 C CNN
+F 0 "#PWR047" H 5925 8175 50  0001 C CNN
 F 1 "GND" H 5925 8275 50  0000 C CNN
 F 2 "" H 5925 8425 50  0001 C CNN
@@
 $EndComp
 $Comp
-L GND #PWR044
+L GND #PWR048
 U 1 1 59CF101D
 P 10700 3975
-F 0 "#PWR044" H 10700 3725 50  0001 C CNN
+F 0 "#PWR048" H 10700 3725 50  0001 C CNN
 F 1 "GND" H 10700 3825 50  0000 C CNN
 F 2 "" H 10700 3975 50  0001 C CNN
@@
 $EndComp
 $Comp
-L GND #PWR045
+L GND #PWR049
 U 1 1 59CFF8CB
 P 4025 4675
-F 0 "#PWR045" H 4025 4425 50  0001 C CNN
+F 0 "#PWR049" H 4025 4425 50  0001 C CNN
 F 1 "GND" H 4025 4525 50  0000 C CNN
 F 2 "" H 4025 4675 50  0001 C CNN
@@
 $EndComp
 $Comp
-L 3V3B #PWR046
+L 3V3B #PWR050
 U 1 1 59D02EA8
 P 13475 1950
-F 0 "#PWR046" H 13475 1800 60  0001 C CNN
+F 0 "#PWR050" H 13475 1800 60  0001 C CNN
 F 1 "3V3B" H 13475 2100 39  0000 C CNN
 F 2 "" H 13475 1950 60  0001 C CNN
@@
 $EndComp
 $Comp
-L GND #PWR047
+L GND #PWR051
 U 1 1 59D0300C
 P 11675 2525
-F 0 "#PWR047" H 11675 2275 50  0001 C CNN
+F 0 "#PWR051" H 11675 2275 50  0001 C CNN
 F 1 "GND" H 11675 2375 50  0000 C CNN
 F 2 "" H 11675 2525 50  0001 C CNN
@@
 $EndComp
 $Comp
-L GND #PWR048
+L GND #PWR052
 U 1 1 59D0DE5D
 P 10400 7425
-F 0 "#PWR048" H 10400 7175 50  0001 C CNN
+F 0 "#PWR052" H 10400 7175 50  0001 C CNN
 F 1 "GND" H 10400 7275 50  0000 C CNN
 F 2 "" H 10400 7425 50  0001 C CNN
@@
 $EndComp
 $Comp
-L GND #PWR049
+L GND #PWR053
 U 1 1 59D0F4EA
 P 10375 7950
-F 0 "#PWR049" H 10375 7700 50  0001 C CNN
+F 0 "#PWR053" H 10375 7700 50  0001 C CNN
 F 1 "GND" H 10375 7800 50  0000 C CNN
 F 2 "" H 10375 7950 50  0001 C CNN
@@
 $EndComp
 $Comp
-L GND #PWR050
+L GND #PWR054
 U 1 1 59D0FC3D
 P 10325 9250
-F 0 "#PWR050" H 10325 9000 50  0001 C CNN
+F 0 "#PWR054" H 10325 9000 50  0001 C CNN
 F 1 "GND" H 10325 9100 50  0000 C CNN
 F 2 "" H 10325 9250 50  0001 C CNN
@@
 $EndComp
 $Comp
-L GND #PWR051
+L GND #PWR055
 U 1 1 59D119A6
 P 10350 8625
-F 0 "#PWR051" H 10350 8375 50  0001 C CNN
+F 0 "#PWR055" H 10350 8375 50  0001 C CNN
 F 1 "GND" H 10350 8475 50  0000 C CNN
 F 2 "" H 10350 8625 50  0001 C CNN
@@
 $EndComp
 $Comp
-L 3V3B #PWR052
+L 3V3B #PWR056
 U 1 1 59D160CA
 P 11850 8000
-F 0 "#PWR052" H 11850 7850 60  0001 C CNN
+F 0 "#PWR056" H 11850 7850 60  0001 C CNN
 F 1 "3V3B" H 11850 8150 39  0000 C CNN
 F 2 "" H 11850 8000 60  0001 C CNN
@@
 35MHz anti alias filter
 $Comp
-L GND #PWR053
+L GND #PWR057
 U 1 1 59CB2384
 P 3675 6475
-F 0 "#PWR053" H 3675 6225 50  0001 C CNN
+F 0 "#PWR057" H 3675 6225 50  0001 C CNN
 F 1 "GND" H 3675 6325 50  0000 C CNN
 F 2 "" H 3675 6475 50  0001 C CNN
@@
 $EndComp
 $Comp
-L GND #PWR054
+L GND #PWR058
 U 1 1 59CE0519
 P 5400 4900
-F 0 "#PWR054" H 5400 4650 50  0001 C CNN
+F 0 "#PWR058" H 5400 4650 50  0001 C CNN
 F 1 "GND" H 5400 4750 50  0000 C CNN
 F 2 "" H 5400 4900 50  0001 C CNN
@@
 CLK
 $Comp
-L +3V3Rpi #PWR055
+L +3V3Rpi #PWR057
 U 1 1 59CFD2A8
-P 5400 3625
-F 0 "#PWR055" H 5375 3400 60  0001 C CNN
-F 1 "+3V3Rpi" H 5425 3825 60  0000 C CNN
-F 2 "" H 5400 3625 60  0001 C CNN
-F 3 "" H 5400 3625 60  0001 C CNN
-	1    5400 3625
+P 5400 3555
+AR Path="/59CFD2A8" Ref="#PWR057"  Part="1"
+AR Path="/59BC4A83/59CFD2A8" Ref="#PWR059"  Part="1"
+F 0 "#PWR059" H 5375 3330 60  0001 C CNN
+F 1 "+3V3Rpi" H 5425 3755 60  0000 C CNN
+F 2 "" H 5400 3555 60  0001 C CNN
+F 3 "" H 5400 3555 60  0001 C CNN
+	1    5400 3555
 	1    0    0    -1
 $EndComp
@@
 Text Label 10600 4650 0    39   ~ 0
 MODE
+Text Label 9725 7150 0    39   ~ 0
+AVDD3
+Text Label 9725 7650 0    39   ~ 0
+CLKVDD
+Text Label 9600 8300 0    39   ~ 0
+AVDD
+Text Label 9600 8950 0    39   ~ 0
+DVDD
+Text Label 5975 4550 0    39   ~ 0
+IOUT_N-
+Text Label 5975 4150 0    39   ~ 0
+IOUT_N+
+Text Label 5925 5950 0    39   ~ 0
+RX+
+Text Label 5950 6350 0    39   ~ 0
+RX-
+Text Notes 13125 2700 0    118  ~ 24
+38.4 MHz
+Text GLabel 5400 3625 2    39   Input ~ 0
+3V3Rpi
 Wire Wire Line
 	5925 7750 6325 7750
@@
 Connection ~ 5925 6550
 Wire Wire Line
-	7475 8250 7475 8300
-Wire Wire Line
-	7475 8300 5925 8300
+	7475 8300 7475 8250
+Wire Wire Line
+	5925 8300 7475 8300
 Connection ~ 5925 8300
 Wire Wire Line
@@
 Connection ~ 11800 2150
 Wire Wire Line
-	12800 2300 12800 2625
-Wire Wire Line
-	12800 2625 11800 2625
+	11800 2625 13240 2625
 Connection ~ 11800 2450
 Wire Wire Line
@@
 	3025 5850 3350 5850
 Wire Wire Line
-	3275 6175 3275 5850
+	3275 5850 3275 6175
 Connection ~ 3275 5850
 Wire Wire Line
@@
 Connection ~ 3675 6050
 Wire Wire Line
-	4400 5900 4400 5850
+	4400 5850 4400 5900
 Connection ~ 4400 5850
 Wire Wire Line
@@
 	4000 5850 4000 6175
 Wire Wire Line
-	4400 6300 4400 6425
+	4400 6425 4400 6300
 Wire Wire Line
 	2625 6425 2625 5950
@@
 	5325 4550 6325 4550
 Wire Wire Line
-	5400 3625 5400 3750
-Wire Wire Line
 	5400 4050 5400 4650
 Wire Wire Line
@@
 Wire Wire Line
 	10575 3975 10700 3975
-Connection ~ 5400 3625
 Connection ~ 6325 3625
 Connection ~ 12800 2150
@@
 Connection ~ 4925 4150
 Connection ~ 5325 4150
-Connection ~ 5400 4050
-Connection ~ 5400 3750
 Wire Wire Line
 	9725 5025 11850 5025
@@
 Connection ~ 10350 8625
 Connection ~ 10375 7950
-Text Label 9725 7150 0    39   ~ 0
-AVDD3
-Text Label 9725 7650 0    39   ~ 0
-CLKVDD
-Text Label 9600 8300 0    39   ~ 0
-AVDD
-Text Label 9600 8950 0    39   ~ 0
-DVDD
-Text Label 5975 4550 0    39   ~ 0
-IOUT_N-
-Text Label 5975 4150 0    39   ~ 0
-IOUT_N+
-Text Label 5925 5950 0    39   ~ 0
-RX+
-Text Label 5950 6350 0    39   ~ 0
-RX-
-Text Notes 13125 2700 0    118  ~ 24
-38.4 MHz
 Wire Wire Line
 	11700 8000 11850 8000
+Wire Wire Line
+	12800 2300 13240 2300
+Wire Wire Line
+	13240 2300 13240 2625
+Connection ~ 11245 8950
+Connection ~ 11275 8295
+Connection ~ 11295 7650
+Connection ~ 11325 7150
+Wire Wire Line
+	5400 3555 5400 3750
 $EndSCHEMATC

Commit message: radioberry beta3
Parts:
- added C438: 100nF, hermeslite:SMD-0603, symbol C_Small
Connections:
- net CLK: now also C438.2; no longer IC401.57 (OSCIN)
- new net: C438.1, IC401.57 (OSCIN)
Changed lines of the file:
@@
 Text GLabel 12900 2450 2    60   Input ~ 0
 CLK
-Text GLabel 6325 3625 0    60   Input ~ 0
+Text GLabel 6050 3625 0    60   Input ~ 0
 CLK
 $Comp
@@
 Wire Wire Line
 	5400 3555 5400 3750
+$Comp
+L C_Small C438
+U 1 1 5BD90CBE
+P 6225 3625
+F 0 "C438" V 6075 3525 50  0000 L CNN
+F 1 "100nF" V 6350 3525 50  0000 L CNN
+F 2 "hermeslite:SMD-0603" H 6225 3625 50  0001 C CNN
+F 3 "" H 6225 3625 50  0001 C CNN
+	1    6225 3625
+	0    1    1    0
+$EndComp
+Wire Wire Line
+	6050 3625 6125 3625
+Connection ~ 6125 3625
 $EndSCHEMATC

Commit message: beta4
Parts:
- C401, C402, C403, C404, C405, C406, C407, C408, C409, C410, C411, C412, C413, C414, C415, C416, C417, C418, C419, C420, C421, C422, C423, C424, C425, C426, C427, C428, C429, C430, C431, C432, C433, C434, C435, C436, C437, C438: symbol C_Small -> hermeslite:C_Small
- D401: symbol DIODESCH2 -> hermeslite:DIODESCH2
- F401, F402: symbol MURATA-FILTER_NFM21C -> Radioberry:MURATA-FILTER_NFM21C
- FB401, FB402, FB403, FB404, FB405, FB406: symbol FB -> hermeslite:FB
- IC401: symbol AD9866_AD9866 -> Radioberry:AD9866_AD9866
- L401, L402: symbol L_Small -> hermeslite:L_Small
- R403: symbol RCL_R-EU_R0805 -> Radioberry:RCL_R-EU_R0805
- T401, T402: symbol PA3GSB_T1-1TDIL -> Radioberry:PA3GSB_T1-1TDIL
- U1: symbol FPGA -> Radioberry:FPGA
- X400: symbol TCXO -> Radioberry:TCXO
- X401, X402: symbol CON-COAX_BU-SMA-H -> Radioberry:CON-COAX_BU-SMA-H
Connections:
- net CLKOUT1: now also U1.53 (CLKOUT1)
