File: hardware/Radioberry-PWR.sch (KiCad schematic (older format))
At the start: 73 parts, among them IC201 LD1117S25, IC202 LD1117S33, IC203 LD1117S33, IC204 LD1117S12, U1 FPGA

Commit message: radioberry v2.0 beta2
Connections:
- net +1V2: now also U1.134 (VCCINT), U1.61 (VCCINT)
- net +2V5: now also C216.1, IC204.3 (IN)
- net 3V3B: no longer C216.1, IC204.3 (IN)
Other:
- note added: "Cyclone 10LP : Possible use : 10CL016 or 10CL025"
- note added: "Supply AD9866"
- note added: "Supply FPGA"
- note removed: "3v3a"
- note removed: "connect to 2,5v???"
- moved on the sheet: C216, C217, C218, C219, C220, IC204, R201

Commit message: beta4
Parts:
- C201, C202, C203, C204, C205, C206, C207, C208, C209, C210, C211, C212, C213, C214, C215, C216, C217, C218, C219, C220, C221, C222, C223, C224, C225, C226, C227, C228, C229, C230, C231, C232, C233, C234, C235, C236, C237, C238, C239, C240, C241, C242, C243, C244, C245, C246, C247, C248, C249, C250, C251, C252, C253, C254, C255, C256, C257, C258, C259: symbol C_Small -> hermeslite:C_Small
- FB201, FB202, FB203, FB204, FB205, FB206, FB207, FB208: symbol FB -> hermeslite:FB
- IC201, IC202, IC203: symbol V-REG_LD117AS33TR -> Radioberry:V-REG_LD117AS33TR
- IC204: symbol V-REG_LD117AS12TR -> Radioberry:V-REG_LD117AS12TR
- R201: symbol RCL_R-EU_R0805 -> Radioberry:RCL_R-EU_R0805
- U1: symbol FPGA -> Radioberry:FPGA
Connections:
- net GND: now also U1.69-UE (ClkOUT1); no longer U1.118 (GND)
