File: hardware/Radioberry.sch (KiCad schematic (older format))
At the start: 4 parts

Commit message: beta4
Parts:
- MH1, MH2, MH3, MH4: symbol TEST_1P -> hermeslite:TEST_1P
Changed lines of the file:
@@
-EESchema Schematic File Version 2
-LIBS:Radioberry
-LIBS:hermeslite
-LIBS:power
-LIBS:Radioberry-cache
-EELAYER 25 0
+EESchema Schematic File Version 4
+EELAYER 30 0
 EELAYER END
 $Descr A4 11693 8268
@@
 Sheet 1 4
 Title "RadioBerry V2.0"
-Date "2017-11-29"
-Rev "beta2"
+Date "2020-10-01"
+Rev "beta4"
 Comp "AppMind"
 Comment1 "PA3GSB"
@@
 $EndSheet
 $Comp
-L TEST_1P MH1
+L hermeslite:TEST_1P MH1
 U 1 1 59CC9E7F
 P 6125 4750
@@
 $EndComp
 $Comp
-L TEST_1P MH2
+L hermeslite:TEST_1P MH2
 U 1 1 59CC9EF6
 P 6300 4750
@@
 $EndComp
 $Comp
-L TEST_1P MH3
+L hermeslite:TEST_1P MH3
 U 1 1 59CC9F32
 P 6475 4750
@@
 $EndComp
 $Comp
-L TEST_1P MH4
+L hermeslite:TEST_1P MH4
 U 1 1 59CC9F63
 P 6650 4750
@@
 $EndComp
 $Comp
-L GND #PWR01
+L hermeslite:GND #PWR01
 U 1 1 59CC9F91
 P 6375 5000
@@
 	6125 4750 6125 4875
 Wire Wire Line
-	6125 4875 6650 4875
+	6125 4875 6300 4875
 Wire Wire Line
 	6300 4750 6300 4875
@@
 Wire Wire Line
 	6375 4875 6375 5000
+Wire Wire Line
+	6300 4875 6375 4875
+Wire Wire Line
+	6375 4875 6475 4875
+Wire Wire Line
+	6475 4875 6650 4875
 $EndSCHEMATC
