File: hardware/Raspberry-GPIO.sch (KiCad schematic (older format))
At the start: 9 parts, among them CN301 DNI, CN302 PINHEAD_PINHD-2X20, U1 FPGA

Commit message: radioberry v2.0 beta2
Parts:
- added R307, R308: DNI, hermeslite:SMD-0603, symbol RCL_R-EU_R0805
Connections:
- net +3V3: now also R307.2, R308.2
- net GND: now also CN302.9
- net IO-11: now also R307.1
- net IO-12: now also R308.1
- net 3V3Rpi: now reaches CN302.1
- no-connect marks 11 -> 9
Other:
- note added: "(internal FPGA pull up to large / avoiding speed problems)"
- note added: "Option pull-ups"
- note added: "Programming pull-ups"
- moved on the sheet: R301, R302, R303, R304

Commit message: beta4
Parts:
- CN301: symbol PINHEAD_PINHD-2X10 -> Radioberry:PINHEAD_PINHD-2X10
- CN302: symbol PINHEAD_PINHD-2X20 -> Radioberry:PINHEAD_PINHD-2X20
- R301, R302, R303, R304, R305, R306, R307, R308: symbol RCL_R-EU_R0805 -> Radioberry:RCL_R-EU_R0805
- U1: symbol FPGA -> Radioberry:FPGA
Changed lines of the file:
@@
-EESchema Schematic File Version 2
-LIBS:Radioberry
-LIBS:hermeslite
-LIBS:power
-LIBS:Radioberry-cache
-EELAYER 25 0
+EESchema Schematic File Version 4
+EELAYER 30 0
 EELAYER END
 $Descr A4 11693 8268
@@
 Sheet 3 4
 Title ""
-Date ""
-Rev "rev 2.0-beta1"
+Date "2020-10-01"
+Rev "beta4"
 Comp "AppMind"
 Comment1 "PA3GSB"
@@
 $EndDescr
 $Comp
-L RCL_R-EU_R0805 R?
+L Radioberry:RCL_R-EU_R0805 R?
 U 1 1 59BD2E97
 P 6610 2030
@@
 $EndComp
 $Comp
-L RCL_R-EU_R0805 R?
+L Radioberry:RCL_R-EU_R0805 R?
 U 1 1 59BD2E9E
 P 6610 2230
@@
 	4400 2550 4500 2650
 $Comp
-L PINHEAD_PINHD-2X10 CN301
+L Radioberry:PINHEAD_PINHD-2X10 CN301
 U 1 1 59BE5672
 P 1900 6150
@@
 Input-Output
 $Comp
-L GND #PWR036
+L hermeslite:GND #PWR036
 U 1 1 59BE8319
 P 1525 6650
@@
 $EndComp
 $Comp
-L GND #PWR037
+L hermeslite:GND #PWR037
 U 1 1 59BE8382
 P 2350 6650
@@
 FPGA-PROGRAMMING
 $Comp
-L GND #PWR038
+L hermeslite:GND #PWR038
 U 1 1 59BF4346
 P 3050 3675
@@
 $EndComp
 $Comp
-L GND #PWR039
+L hermeslite:GND #PWR039
 U 1 1 59BF4427
 P 8475 1625
@@
 $EndComp
 $Comp
-L FPGA U1
+L Radioberry:FPGA U1
 U 3 1 59BF65A5
 P 4200 6900
@@
 SPI-0
 $Comp
-L FPGA U1
+L Radioberry:FPGA U1
 U 2 1 59BF8246
 P 9225 3800
@@
 	3600 6950 3700 6850
 $Comp
-L FPGA U1
+L Radioberry:FPGA U1
 U 1 1 59C96E6B
 P 9275 2525
@@
 CE1_SPI0
 $Comp
-L +3V3 #PWR040
+L hermeslite:+3V3 #PWR040
 U 1 1 59CA01AB
 P 7110 1930
@@
 NSTATUS
 $Comp
-L +3V3 #PWR041
+L hermeslite:+3V3 #PWR041
 U 1 1 59CA284E
 P 2475 5650
@@
 $EndComp
 $Comp
-L FPGA U1
+L Radioberry:FPGA U1
 U 4 1 59CA3DF2
 P 9000 6150
@@
 $EndComp
 $Comp
-L +5V #PWR307
+L Radioberry:+5V #PWR307
 U 1 1 59CDA96D
 P 4000 1300
@@
 $EndComp
 $Comp
-L +5V #PWR301
+L Radioberry:+5V #PWR301
 U 1 1 59CFABA8
 P 1450 5675
@@
 $EndComp
 $Comp
-L +3V3Rpi #PWR042
+L Radioberry:+3V3Rpi #PWR042
 U 1 1 59CFC626
 P 2555 1350
@@
 NoConn ~ 3375 2650
 $Comp
-L PINHEAD_PINHD-2X20 CN302
+L Radioberry:PINHEAD_PINHD-2X20 CN302
 U 1 1 59BE4EE2
 P 3075 2250
@@
 IO-13
 $Comp
-L RCL_R-EU_R0805 R?
+L Radioberry:RCL_R-EU_R0805 R?
 U 1 1 59D7BD3F
 P 6655 5085
@@
 $EndComp
 $Comp
-L RCL_R-EU_R0805 R?
+L Radioberry:RCL_R-EU_R0805 R?
 U 1 1 59D7BAFD
 P 6645 4850
@@
 GPCLK2
 $Comp
-L RCL_R-EU_R0805 R?
+L Radioberry:RCL_R-EU_R0805 R?
 U 1 1 59E4A415
 P 6625 5700
@@
 $EndComp
 $Comp
-L RCL_R-EU_R0805 R?
+L Radioberry:RCL_R-EU_R0805 R?
 U 1 1 59E4A48A
 P 6625 5950
@@
 NoConn ~ 8850 4600
 $Comp
-L RCL_R-EU_R0805 R?
+L Radioberry:RCL_R-EU_R0805 R?
 U 1 1 5A10530B
 P 6675 3425
@@
 IO-12
 $Comp
-L +3V3 #PWR043
+L hermeslite:+3V3 #PWR043
 U 1 1 5A116B28
 P 7125 3280
@@
 Programming pull-ups
 $Comp
-L +3V3 #PWR044
+L hermeslite:+3V3 #PWR044
 U 1 1 5A173804
 P 7220 4770
@@
 SDA
 $Comp
-L RCL_R-EU_R0805 R?
+L Radioberry:RCL_R-EU_R0805 R?
 U 1 1 5A105358
 P 6675 3675
@@
 $EndComp
 $Comp
-L PWR_FLAG #FLG045
+L power:PWR_FLAG #FLG045
 U 1 1 5A2114A8
 P 995 1045
@@
 $EndComp
 $Comp
-L +3V3Rpi #PWR046
+L Radioberry:+3V3Rpi #PWR046
 U 1 1 5A2114D8
 P 995 1095
@@
 $EndComp
 Wire Wire Line
-	2425 1750 2425 3650
-Wire Wire Line
-	2425 3650 3725 3650
-Wire Wire Line
-	3725 3650 3725 1550
+	2425 1750 2425 2550
+Wire Wire Line
+	2425 3650 3050 3650
+Wire Wire Line
+	3725 3650 3725 2950
 Connection ~ 2425 2550
-Connection ~ 2425 1750
 Connection ~ 2425 3250
 Connection ~ 3725 2950
@@
 Wire Wire Line
 	6810 2030 7110 2030
-Connection ~ 6810 2030
 Connection ~ 7110 2030
-Connection ~ 6810 2230
 Wire Wire Line
 	3775 1450 3375 1450
 Wire Wire Line
-	3375 1350 4000 1350
+	3375 1350 3775 1350
 Wire Wire Line
 	3775 1350 3775 1450
 Connection ~ 3775 1350
-Wire Bus Line
-	1625 2350 1625 4275
-Wire Bus Line
-	4500 2550 4500 4275
-Wire Bus Line
-	6125 7075 1075 7075
 Wire Wire Line
 	1700 5950 1175 5950
@@
 Wire Wire Line
 	2200 5850 2725 5850
-Wire Bus Line
-	1075 7075 1075 5950
-Wire Bus Line
-	2825 5950 2825 7075
 Wire Wire Line
 	2200 5950 2725 5950
@@
 	2875 1950 1500 1950
 Wire Bus Line
-	1400 2050 1400 4625
-Wire Bus Line
 	1400 4625 5050 4625
 Wire Wire Line
@@
 	8675 2425 9125 2425
 Wire Bus Line
-	8575 1925 8575 2925
-Wire Bus Line
 	8575 2925 9700 2925
 Wire Wire Line
 	9125 1625 8475 1625
 Wire Wire Line
-	9125 1325 9125 1625
+	9125 1325 9125 1425
 Connection ~ 9125 1425
 Connection ~ 9125 1525
 Connection ~ 9125 1625
-Connection ~ 9125 1325
-Connection ~ 8475 1625
 Wire Wire Line
 	8675 3300 9125 3300
@@
 	8675 3700 9125 3700
 Wire Bus Line
-	8575 3400 8575 4175
-Wire Bus Line
 	8575 4175 9825 4175
 Wire Wire Line
@@
 Wire Wire Line
 	5600 6850 6025 6850
-Wire Bus Line
-	3600 6250 3600 7075
-Wire Bus Line
-	3600 7075 3575 7075
 Wire Wire Line
 	1175 5850 1700 5850
 Wire Wire Line
-	7110 1930 7110 2230
+	7110 1930 7110 2030
 Wire Wire Line
 	2875 3250 2425 3250
@@
 Wire Wire Line
 	8775 5000 8850 5000
-Connection ~ 6410 2030
-Connection ~ 6410 2230
 Wire Wire Line
 	3050 3675 3050 3650
 Connection ~ 3050 3650
-Wire Bus Line
-	6125 6450 6125 7075
 Wire Wire Line
 	1700 6550 1550 6550
@@
 	6425 5700 6200 5700
 Wire Wire Line
-	6200 5950 6425 5950
-Wire Wire Line
 	6825 5700 7075 5700
 Wire Wire Line
@@
 Wire Wire Line
 	6160 2230 6410 2230
-Connection ~ 6825 5950
-Connection ~ 6820 5695
-Connection ~ 6430 5705
-Connection ~ 6420 5950
 Wire Wire Line
 	6455 5085 6200 5085
@@
 	6845 4850 7220 4850
 Wire Wire Line
-	7220 4770 7220 5085
+	7220 4770 7220 4850
 Wire Wire Line
 	7220 5085 6855 5085
@@
 	6875 3425 7125 3425
 Wire Wire Line
-	7125 3280 7125 3675
+	7125 3280 7125 3425
 Wire Wire Line
 	7125 3675 6875 3675
@@
 	995  1045 995  1095
 Wire Wire Line
-	2415 1350 2875 1350
+	2415 1350 2555 1350
 Connection ~ 2555 1350
 Text GLabel 2415 1350 0    39   Input ~ 0
 3V3Rpi
+Wire Wire Line
+	2425 2550 2425 3250
+Wire Wire Line
+	2425 3250 2425 3650
+Wire Wire Line
+	3725 2950 3725 2750
+Wire Wire Line
+	3725 2750 3725 2250
+Wire Wire Line
+	3725 2250 3725 1950
+Wire Wire Line
+	3725 1950 3725 1550
+Wire Wire Line
+	7110 2030 7110 2230
+Wire Wire Line
+	3775 1350 4000 1350
+Wire Wire Line
+	9125 1425 9125 1525
+Wire Wire Line
+	9125 1525 9125 1625
+Wire Wire Line
+	3050 3650 3725 3650
+Wire Wire Line
+	7220 4850 7220 5085
+Wire Wire Line
+	7125 3425 7125 3675
+Wire Wire Line
+	2555 1350 2875 1350
+Wire Bus Line
+	1075 7075 6125 7075
+Wire Wire Line
+	6200 5950 6425 5950
+Wire Bus Line
+	4500 2550 4500 4275
+Wire Bus Line
+	1625 2350 1625 4275
+Wire Bus Line
+	1400 2050 1400 4625
+Wire Bus Line
+	8575 1925 8575 2925
+Wire Bus Line
+	8575 3400 8575 4175
+Wire Bus Line
+	1075 5950 1075 7075
+Wire Bus Line
+	2825 5950 2825 7075
+Wire Bus Line
+	6125 6450 6125 7075
+Wire Bus Line
+	3600 6250 3600 7075
 $EndSCHEMATC
