File: hardware/radio/Radioberry-Frontend.sch (KiCad schematic (older format))
At the start: 57 parts, among them IC401 AD9866, T401 1:1, T402 8:1, U1 FPGA, X400 TCXO, X401 SMA, X402 SMA

Commit message: beta5 special thanks to VU2UPX
Parts:
- C401, C402, C409, C410, C411, C412, C414, C415, C416, C417, C418, C419, C420, C421, C422, C423, C424, C425, C426, C427, C428, C429, C430, C431, C432, C433, C434, C435, C436, C437, C438: footprint hermeslite:SMD-0603 -> +VU2UPX_FOOTPRINT:C_0603_1608Metric_Pad1.08x0.95mm_HandSolder
- C403, C404, C405, C406, C407: footprint hermeslite:SMD-0805 -> +VU2UPX_FOOTPRINT:C_0805_2012Metric_Pad1.18x1.45mm_HandSolder
- C408: footprint hermeslite:SMD-1206 -> Capacitor_SMD:C_1206_3216Metric_Pad1.33x1.80mm_HandSolder
- C413: footprint hermeslite:SMD-0805 -> +VU2UPX_FOOTPRINT:C_0603_1608Metric_Pad1.08x0.95mm_HandSolder
- D401: footprint hermeslite:SOD323 -> +VU2UPX_FOOTPRINT:SOD323
- F401, F402: footprint Radioberry:MURATA-FILTER_NFM21C -> +VU2UPX_FOOTPRINT:MURATA-FILTER_NFM21C
- FB401, FB402, FB403, FB404, FB405, FB406: footprint hermeslite:SMD-0603 -> +VU2UPX_FOOTPRINT:VU2UPX_0603_HandSolder
- L401, L402: footprint hermeslite:SMD-0805 -> +VU2UPX_FOOTPRINT:VU2UPX_0805__HandSolder
- R403: footprint hermeslite:SMD-0603 -> +VU2UPX_FOOTPRINT:R_0603_1608Metric_Pad0.98x0.95mm_HandSolder
- T401, T402: footprint hermeslite:TR1-1 -> +VU2UPX_FOOTPRINT:TR1-1
- X400: footprint hermeslite:TCXO -> +VU2UPX_FOOTPRINT:TCXO
