File: hardware/radio/Radioberry-PWR.sch (KiCad schematic (older format))
At the start: 73 parts, among them IC201 LD1117S25, IC202 LD1117S33, IC203 LD1117S33, IC204 LD1117S12, U1 FPGA

Commit message: beta5 special thanks to VU2UPX
Parts:
- C201, C202, C203, C204, C205, C206, C207, C208, C209, C210, C211, C212, C216, C217, C218, C219, C221, C222, C223, C224, C225, C226, C227, C228, C229, C230, C231, C232, C233, C234, C235, C236, C237, C238, C239, C240, C241, C242, C243, C244, C245, C246, C247, C248, C249, C250, C251, C252, C253, C254, C255, C256, C257, C258, C259: footprint hermeslite:SMD-0603 -> +VU2UPX_FOOTPRINT:C_0603_1608Metric_Pad1.08x0.95mm_HandSolder
- C213, C214, C215, C220: footprint hermeslite:SMD-1210 -> Capacitor_SMD:C_1210_3225Metric_Pad1.33x2.70mm_HandSolder
- FB201, FB202, FB203, FB204, FB205, FB206, FB207, FB208: footprint hermeslite:SMD-0603 -> +VU2UPX_FOOTPRINT:VU2UPX_0603_HandSolder
