File: hardware/radio/Raspberry-GPIO.sch (KiCad schematic (older format))
At the start: 11 parts, among them CN301 DNI, CN302 PINHEAD_PINHD-2X20, U1 FPGA

Commit message: beta5 special thanks to VU2UPX
Parts:
- R301, R302, R303, R304, R305, R306, R307, R308: footprint hermeslite:SMD-0603 -> +VU2UPX_FOOTPRINT:R_0603_1608Metric_Pad0.98x0.95mm_HandSolder
Changed lines of the file:
@@
 Sheet 3 4
 Title ""
-Date "2020-10-01"
-Rev "beta4"
+Date "2021-04-21"
+Rev "beta5"
 Comp "AppMind"
 Comment1 "PA3GSB"
@@
 F 0 "R301" H 6460 2089 70  0000 L BNN
 F 1 "10K" H 6760 2099 70  0000 L BNN
-F 2 "hermeslite:SMD-0603" H 6600 1820 65  0001 L TNN
+F 2 "+VU2UPX_FOOTPRINT:R_0603_1608Metric_Pad0.98x0.95mm_HandSolder" H 6600 1820 65  0001 L TNN
 F 3 "" H 6610 2030 60  0001 C CNN
 	1    6610 2030
@@
 F 0 "R302" H 6460 2289 70  0000 L BNN
 F 1 "10K" H 6760 2299 70  0000 L BNN
-F 2 "hermeslite:SMD-0603" H 6600 2020 65  0001 L TNN
+F 2 "+VU2UPX_FOOTPRINT:R_0603_1608Metric_Pad0.98x0.95mm_HandSolder" H 6600 2020 65  0001 L TNN
 F 3 "" H 6610 2230 60  0001 C CNN
 	1    6610 2230
@@
 F 0 "R304" H 6505 5144 70  0000 L BNN
 F 1 "DNI" H 6805 5154 70  0000 L BNN
-F 2 "hermeslite:SMD-0603" H 6645 4875 65  0001 L TNN
+F 2 "+VU2UPX_FOOTPRINT:R_0603_1608Metric_Pad0.98x0.95mm_HandSolder" H 6645 4875 65  0001 L TNN
 F 3 "" H 6655 5085 60  0001 C CNN
 F 4 "GENERIC" H 6655 5085 60  0001 C CNN "Option"
@@
 F 0 "R303" H 6495 4909 70  0000 L BNN
 F 1 "DNI" H 6795 4919 70  0000 L BNN
-F 2 "hermeslite:SMD-0603" H 6635 4640 65  0001 L TNN
+F 2 "+VU2UPX_FOOTPRINT:R_0603_1608Metric_Pad0.98x0.95mm_HandSolder" H 6635 4640 65  0001 L TNN
 F 3 "" H 6645 4850 60  0001 C CNN
 F 4 "GENERIC" H 6645 4850 60  0001 C CNN "Option"
@@
 F 0 "R305" H 6475 5759 70  0000 L BNN
 F 1 "DNI" H 6775 5769 70  0000 L BNN
-F 2 "hermeslite:SMD-0603" H 6615 5490 65  0001 L TNN
+F 2 "+VU2UPX_FOOTPRINT:R_0603_1608Metric_Pad0.98x0.95mm_HandSolder" H 6615 5490 65  0001 L TNN
 F 3 "" H 6625 5700 60  0001 C CNN
 F 4 "GENERIC" H 6625 5700 60  0001 C CNN "Option"
@@
 F 0 "R306" H 6475 6009 70  0000 L BNN
 F 1 "DNI" H 6775 6019 70  0000 L BNN
-F 2 "hermeslite:SMD-0603" H 6615 5740 65  0001 L TNN
+F 2 "+VU2UPX_FOOTPRINT:R_0603_1608Metric_Pad0.98x0.95mm_HandSolder" H 6615 5740 65  0001 L TNN
 F 3 "" H 6625 5950 60  0001 C CNN
 F 4 "GENERIC" H 6625 5950 60  0001 C CNN "Option"
@@
 F 0 "R308" H 6525 3500 70  0000 L BNN
 F 1 "DNI" H 6825 3325 70  0000 L BNN
-F 2 "hermeslite:SMD-0603" H 6665 3215 65  0001 L TNN
+F 2 "+VU2UPX_FOOTPRINT:R_0603_1608Metric_Pad0.98x0.95mm_HandSolder" H 6665 3215 65  0001 L TNN
 F 3 "" H 6675 3425 60  0001 C CNN
 F 4 "GENERIC" H 6675 3425 60  0001 C CNN "Option"
@@
 F 0 "R307" H 6475 3525 70  0000 L BNN
 F 1 "DNI" H 6825 3575 70  0000 L BNN
-F 2 "hermeslite:SMD-0603" H 6665 3465 65  0001 L TNN
+F 2 "+VU2UPX_FOOTPRINT:R_0603_1608Metric_Pad0.98x0.95mm_HandSolder" H 6665 3465 65  0001 L TNN
 F 3 "" H 6675 3675 60  0001 C CNN
 F 4 "GENERIC" H 6675 3675 60  0001 C CNN "Option"
